Commit message: “firstcommit”

File: src/install/july_9/share/july_9/robot_description/robot_core.xacro (robot description, xacro)
@@ -18,4 +18,11 @@
     <link name="base_link">
     </link>
+    <link name="base_footprint">
+    </link>
+    <joint name="base_footprint_joint" type="fixed">
+        <parent link="base_link"/>
+        <child link="base_footprint"/>
+        <origin xyz="0.0 0.0 0.0" rpy="0.0 0.0 0.0"/>
+    </joint>
     <!-- base link to chassis-->
     <joint name="base_chassis" type="fixed">
@@ -28,5 +35,5 @@
         <visual>
             <geometry>
-                <cylinder radius="0.06" length="0.03"/>
+                <cylinder radius="0.08" length="0.03"/>
             </geometry>
             <material name="yellow">
@@ -36,8 +43,8 @@
         <collision>
             <geometry>
-                <cylinder radius="0.06" length="0.03"/>
+                <cylinder radius="0.08" length="0.03"/>
             </geometry>
         </collision>
-        <xacro:inertial_cylinder mass="0.1"  length="0.03" radius="0.06">
+        <xacro:inertial_cylinder mass="0.1"  length="0.03" radius="0.08">
             <origin xyz="0 0 0" rpy="0 0 0"/>
         </xacro:inertial_cylinder>
@@ -50,5 +57,5 @@
         <parent link="base_link"/> <!--here left wheel linked base link becoz of the base link at the centre of the rotation-->
         <child link="left_wheel"/>
-        <origin xyz="0.0 0.115 0.0" rpy="-${pi/2} 0.0 0.0"/>
+        <origin xyz="0.0 0.115 0.0" rpy="${pi/2} 0.0 0.0"/>
         <axis xyz="0.0 0.0 1"/>
     </joint>
@@ -57,5 +64,5 @@
         <visual>
             <geometry>
-                <cylinder radius="0.06" length="0.03"/>
+                <cylinder radius="0.08" length="0.03"/>
             </geometry>
             <material name="yellow">
@@ -65,8 +72,8 @@
         <collision>
             <geometry>
-                <cylinder radius="0.06" length="0.03"/>
+                <cylinder radius="0.08" length="0.03"/>
             </geometry>
         </collision>
-        <xacro:inertial_cylinder mass="0.1"  length="0.03" radius="0.06">
+        <xacro:inertial_cylinder mass="0.1"  length="0.03" radius="0.08">
             <origin xyz="0 0 0" rpy="0 0 0"/>
         </xacro:inertial_cylinder>
@@ -79,5 +86,5 @@
         <parent link="base_link"/> <!--here left wheel linked base link becoz of the base link at the centre of the rotation-->
         <child link="right_wheel"/>
-        <origin xyz="0.0 -0.115 0.0" rpy="${pi/2} 0.0 0.0"/>
+        <origin xyz="0.0 -0.115 0.0" rpy="-${pi/2} 0.0 0.0"/>
         <axis xyz="0.0 0.0 -1"/>
     </joint>
@@ -86,5 +93,5 @@
         <visual>
             <geometry>
-                <sphere radius="0.03"/>
+                <sphere radius="0.04"/>
             </geometry>
             <material name="black"/>
@@ -92,8 +99,8 @@
         <collision>
             <geometry>
-                <sphere radius="0.03"/>
+                <sphere radius="0.04"/>
             </geometry>
         </collision>
-        <xacro:inertial_sphere mass="0.35" radius="0.03">
+        <xacro:inertial_sphere mass="0.35" radius="0.04">
             <origin xyz="0 0 0" rpy="0 0 0"/>
         </xacro:inertial_sphere>
@@ -108,5 +115,5 @@
         <parent link="chassis"/>
         <child link="caster_wheel"/>
-        <origin xyz="0.180 0.0 -0.03" rpy="0.0 0.0 0.0"/>
+        <origin xyz="0.180 0.0 -0.04" rpy="0.0 0.0 0.0"/>
     </joint>
 </robot>
